File: Board/TimTime.kicad_pcb (KiCad board)
At the start: 4 copper layers, 58.2 x 32.3 mm, 61 parts, among them IC1 MCP73834-CNI_MF, IC2 LT1761ES5-2.8#TRMPBF, IC3 LTC1844ES5-3.3#TRPBF, J1 USB4085-GF-A_REVA, J2 SJ1-3523NG, J3 Conn_01x04, J4 Conn_01x06, J5 Conn_01x02, J6 Conn_01x02, U1 STM32L433CCTx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

Commit message: V01 Gerbers
Parts:
- added G***: LOGO, Slate_Logo:Slate_Logo_01_Back_Silk, F.Cu at (139.6, 103.8)
- H1, H2, H3, H4: footprint MountingHole:MountingHole_2.7mm_M2.5_Pad_Via -> MountingHole:MountingHole_3.2mm_M3_Pad_Via
- moved R8 2.63 mm to (123.1, 95.4)
- moved R14 1.69 mm to (162.1, 98.3), turned to 270 degrees
- moved J5 1.02 mm to (119.6, 96.4)
- moved H1 0.54 mm to (114.2, 93.0)
- moved H2 0.54 mm to (164.7, 93.0)
- moved H3 0.54 mm to (164.7, 117.6)
- moved H4 0.54 mm to (114.2, 117.6)
Routing:
- net Net-(D1-Pad1): track 2.72 -> 5.68 mm
- net +BATT: track 60.6 -> 59.2 mm
Other:
- board text added: "TimTime Lockit V1.0 Rev. A"
- board text removed: "TimTime Lockit Rev. A-001"
