File: Board/TimTime.kicad_pcb (KiCad board)
At the start: 4 copper layers, 58.2 x 32.3 mm, 62 parts, among them IC1 MCP73834-CNI_MF, IC2 LT1761ES5-2.8#TRMPBF, IC3 LTC1844ES5-3.3#TRPBF, J1 USB4085-GF-A_REVA, J2 SJ1-3523NG, J3 Conn_01x04, J4 Conn_01x06, J5 Conn_01x02, J6 Conn_01x02, U1 STM32L433CCTx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

Commit message: V01B Board
Parts:
- removed D2: DIODE, Diode_SMD:D_SOD-123
- removed H1: MountingHole_Pad, MountingHole:MountingHole_3.2mm_M3_Pad_Via
- added C19: 100nF, Capacitor_SMD:C_0603_1608Metric_Pad1.08x0.95mm_HandSolder, F.Cu at (140.5, 114.4)
- added U3: USBLC6-2SC6, Package_TO_SOT_SMD:SOT-23-6, B.Cu at (119.4, 105.7)
- C1, C10, C11, C12, C14, C15, C16, C3, C4, C5, C6, C7, C8, C9: footprint Capacitor_SMD:C_0603_1608Metric_Pad1.05x0.95mm_HandSolder -> Capacitor_SMD:C_0603_1608Metric_Pad1.08x0.95mm_HandSolder
- C13: value 12uF -> 10uF; footprint Capacitor_SMD:C_0603_1608Metric_Pad1.05x0.95mm_HandSolder -> Capacitor_SMD:C_0603_1608Metric_Pad1.08x0.95mm_HandSolder
- IC3: footprint LT1761ES5-2.8#TRMPBF:SOT95P280X100-5N -> LT1761ES5-2:SOT95P280X100-5N
- R1, R12, R13, R14, R15, R16, R17, R18, R19, R2, R20, R3, R4, R5, R6, R7: footprint Resistor_SMD:R_0603_1608Metric_Pad1.05x0.95mm_HandSolder -> Resistor_SMD:R_0603_1608Metric_Pad0.98x0.95mm_HandSolder
- R10, R11: value 0 -> 10K; footprint Resistor_SMD:R_0603_1608Metric_Pad1.05x0.95mm_HandSolder -> Resistor_SMD:R_0603_1608Metric_Pad0.98x0.95mm_HandSolder
- R8, R9: value 30 -> 60; footprint Resistor_SMD:R_0603_1608Metric_Pad1.05x0.95mm_HandSolder -> Resistor_SMD:R_0603_1608Metric_Pad0.98x0.95mm_HandSolder
- S1, S2, S4: value PTS647SM70SMTR2LFS -> SKPMBHE010; footprint PTS647SM70SMTR2LFS:PTS647SM38SMTR2LFS -> SKPMBHE010:SKPMBHE010
- Y1: footprint 7P-25.000MBP-T:7P25000MBPT -> 7P-25:7P25000MBPT
- moved S2 18.9 mm to (157.2, 96.0), turned to 0 degrees
- moved R14 11.2 mm to (151.0, 96.1), turned to 180 degrees
- moved S1 9.97 mm to (160.5, 105.2), turned to 90 degrees
- moved S4 9.81 mm to (157.2, 114.5), turned to 0 degrees
- moved R4 9.29 mm to (162.6, 111.6), turned to -90 degrees
- moved J5 7.50 mm to (112.2, 95.7)
- moved R15 2.04 mm to (151.0, 115.7)
- moved C14 1.17 mm to (129.3, 109.4), turned to 0 degrees
- moved J2 0.97 mm to (165.0, 105.2)
Connections:
- C14 pad 1: GND -> +3V3
- C14 pad 2: Net-(C14-Pad2) -> GND
- IC2 pad 4: Net-(C14-Pad2) -> unconnected-(IC2-Pad4)
- J1 pad A8: Net-(J1-PadA8) -> unconnected-(J1-PadA8)
- J1 pad B8: Net-(J1-PadB8) -> unconnected-(J1-PadB8)
- J2 pad 3: Net-(J2-Pad3) -> unconnected-(J2-Pad3)
- R10 pad 2: Net-(D2-Pad2) -> TC_OUT
- S1 pad 1: +2V8 -> BTN_C
- S2 pad 1: +2V8 -> BTN_A
- S4 pad 1: +2V8 -> BTN_B
- U1 pad 11: Net-(U1-Pad11) -> unconnected-(U1-Pad11)
- U1 pad 14: Net-(U1-Pad14) -> unconnected-(U1-Pad14)
- U1 pad 16: Net-(U1-Pad16) -> unconnected-(U1-Pad16)
- U1 pad 17: Net-(U1-Pad17) -> unconnected-(U1-Pad17)
- U1 pad 18: Net-(U1-Pad18) -> unconnected-(U1-Pad18)
- U1 pad 20: Net-(U1-Pad20) -> unconnected-(U1-Pad20)
- U1 pad 26: Net-(U1-Pad26) -> unconnected-(U1-Pad26)
- U1 pad 27: Net-(U1-Pad27) -> unconnected-(U1-Pad27)
- U1 pad 28: Net-(U1-Pad28) -> unconnected-(U1-Pad28)
- U1 pad 3: Net-(U1-Pad3) -> unconnected-(U1-Pad3)
- U1 pad 38: Net-(U1-Pad38) -> unconnected-(U1-Pad38)
- U1 pad 4: Net-(U1-Pad4) -> unconnected-(U1-Pad4)
- U1 pad 40: Net-(U1-Pad40) -> unconnected-(U1-Pad40)
- U1 pad 41: Net-(U1-Pad41) -> unconnected-(U1-Pad41)
- U1 pad 44: Net-(U1-Pad44) -> GND
- U1 pad 6: Net-(U1-Pad6) -> unconnected-(U1-Pad6)
- U2 pad 4: Net-(U2-Pad4) -> unconnected-(U2-Pad4)
Routing:
- net Net-(D2-Pad2): track 22.8 -> 0.00 mm
- net +BATT: track 59.2 -> 74.5 mm
- net +3V3: track 9.54 -> 23.3 mm, vias 0 -> 1
- net BTN_C: track 36.7 -> 26.2 mm
- net NRST: track 20.3 -> 29.4 mm
- net GND: track 92.5 -> 100.7 mm, vias 50 -> 54
- net +2V8: track 50.9 -> 42.8 mm
- net TC_OUT: track 11.8 -> 18.0 mm
- net BTN_B: track 23.6 -> 17.5 mm
- net USB_D+: track 21.3 -> 19.1 mm
- net USB_D-: track 20.9 -> 19.0 mm
- net Net-(C14-Pad2): track 1.81 -> 0.00 mm
- net BTN_A: track 41.3 -> 39.5 mm
- net STAT1: track 19.4 -> 20.4 mm
- net STAT2: track 20.7 -> 21.6 mm
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Other:
- net class Default removed
- rule pad_to_mask_clearance: 0.05 -> 0
- board text added: "+2V8"
- board text added: "SCL"
- board text added: "SDA"
- board text added: "TimTime Lockit V1.0 Rev. B"
- board text added: "V"
- board text removed: "TimTime Lockit V1.0 Rev. A"
